File: hardware/KiCad_files/furubot_R2.kicad_pcb (KiCad board)
At the start: 2 copper layers, 55 x 110.1 mm, 126 parts, among them IC1 ULN2803, U1 CONN_01X04, U2 ESP01, U3 CONN_01X04, U4 CONN_01X04, U5 CONN_01X04, U6 LM1117-SOT, X1 Screw_Terminal_1x02

Commit message: Actualización de hardware
Parts:
- ?: moved to B.Cu
- R3: value 10K -> 10K
- R8.1: value 1K -> 1K
- S1.1, S2.1, S3.1, S4.1, S5.1: footprint Switch:SW_PUSH_6mm -> Buttons_Switches_ThroughHole:SW_PUSH_6mm
- moved ? 37.9 mm to (143.9, 143.8)
- moved ? 4.30 mm to (138.3, 136.8)
- moved GND 2.98 mm to (144.3, 54.6)
Routing:
- net /S1: track 44.8 -> 54.2 mm
- net /VIN: track 50.4 -> 59.4 mm
- net /S2: track 61.6 -> 70.4 mm
- net /S5: track 43.6 -> 51.9 mm
- net /S4: track 27.8 -> 35.4 mm
- net /S3: track 74.1 -> 81.6 mm
- net /RAW: track 103.6 -> 99.5 mm
- net Net-(F1-Pad1): track 24.7 -> 26.4 mm
- net /RX: track 27.1 -> 26.2 mm
- net GND: track 19.3 -> 20.0 mm
Other:
- board text added: "Based on: Escornabot.com"
